Commit message: Resolved body issue

File: my_rb1_description/urdf/my_rb1_robot.urdf (robot description, URDF)
Before this commit: robot rb1 robot, 7 links, 6 joints
Links:
- added link body, mass 25; collision cylinder length=0.3 radius=0.25; visual cylinder length=0.3 radius=0.25
- link base_link: mass 25 -> None; geometry 
Joints:
- added joint body_joint: type fixed, parent base_link, child body, origin xyz=0 0 0
